File: Boards/ESP Base Board V1/ESP Base Board V1.kicad_sch (KiCad schematic)
At the start: 16 parts, among them J3 Conn_01x15, J4 Conn_01x15, SW1 RESET

Commit message: Initial Commit
Other:
- moved on the sheet: A0, A1, D0, D1, D10, D11, D2, D3, I2C1, I2C2, J3, J4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
