File: NE555 Timer IC Projects/BATTERY LOW INDIATOR 555/BATTERY LOW INDIATOR 555.kicad_sch (KiCad schematic)
At the start: 16 parts, among them J1 BATTERY, U1 LM555xM, U2 LM393

Commit message: Initial Commit
Other:
- moved on the sheet: BZ1, C1, C2, C3, D1, J1, R1, R2, R3, R4, R5, R6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
