File: NE555 Timer IC Projects/HOME CONTROLLER 555/HOME CONTROLLER 555.kicad_sch (KiCad schematic)
At the start: 52 parts, among them J1 FAN, J2 PIR CONTROLLER, J3 POWER SUPPLY, J4 LIGHT, J5 Conn_01x06, J6 Conn_01x06, K1 SANYOU_SRD_Form_A, K2 SANYOU_SRD_Form_A, K3 SANYOU_SRD_Form_A, Q1 AO3400A, Q2 AO3400A, Q3 AO3400A, SW1 SW_Push, SW2 SW_Push, U1 ESP32-WROOM-32, U2 LM555xM, U3 LM393, U4 LM358, U6 AMS1117-3.3, U7 LM35-LP

Commit message: Initial Commit
Other:
- moved on the sheet: C1, C2, C3, C4, C5, C6, C7, C8, D1, D2, D3, D4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
