File: NE555 Timer IC Projects/LED FLASH 555/LED FLASH 555.kicad_sch (KiCad schematic)
At the start: 8 parts, among them U1 LM555xM

Commit message: Initial Commit
Other:
- moved on the sheet: D1, R1, R2, RV1
