File: Sensors/IR sensor/IR sensor.kicad_pcb (KiCad board)
At the start: 2 copper layers, 10 parts, among them J1 Conn_01x04, U1 LM358

Commit message: Initial Commit
Routing:
- net GND: track 0.00 -> 45.9 mm
- net Net-(D2-K): track 0.00 -> 44.7 mm
- net VCC: track 0.00 -> 39.1 mm, vias 0 -> 2
- net Net-(D3-K): track 0.00 -> 27.1 mm
- net Net-(U1A--): track 0.00 -> 20.6 mm
- net Net-(D1-A): track 0.00 -> 12.3 mm
- net Net-(D3-A): track 0.00 -> 11.2 mm
Other:
- board outline added: 22.5 x 23 mm
