File: Sensors/IR sensor/IR sensor.kicad_sch (KiCad schematic)
At the start: 10 parts, among them J1 Conn_01x04, U1 LM358

Commit message: Initial Commit
Other:
- moved on the sheet: C1, D1, D2, D3, J1, R1, R2, R3, RV1, U1A, U1C
