File: Sensors/Joy Stick V2/Joy Stick V2.kicad_sch (KiCad schematic)
At the start: 65 parts, among them J1 USB_C_Receptacle_USB2.0_14P, J2 Conn_01x02, J3 Micro_SD_Card_Det_Hirose_DM3AT, M1 Motor_DC, Q1 AO3400A, SW1 SW_SPST, U1 CR2013-MI2120, U2 ESP32-WROOM-32, U3 CH340C, U4 AMS1117-3.3, U5 LM386, U6 TP4056-42-ESOP8, X1 SW_Push, Y1 SW_Push

Commit message: Initial Commit
Other:
- moved on the sheet: J3, R1, U2
