File: Sensors/LDR2/LDR2.kicad_sch (KiCad schematic)
At the start: 11 parts, among them J1 Conn_01x04, U1 LM358

Commit message: Initial Commit
Other:
- moved on the sheet: C1, D1, D2, R1, R3, RV1, U1B
